Commit message: sync localhost and github

File: aurmr/src/tahoma_api/tahoma_info/tahoma.urdf (robot description, URDF)
Before this commit: robot tahoma, 71 links, 70 joints
Links:
- link arm_upper_arm_link: geometry collision mesh filename=package://ur_description/meshes/ur16e/collision/upperarm.stl; visual box size=0.1 0.1 0.1
Joints:
- joint gripper_finger_joint: type revolute -> fixed
- joint gripper_left_inner_finger_joint: type revolute -> fixed
- joint gripper_left_inner_knuckle_joint: type revolute -> fixed
- joint gripper_right_finger_joint: type revolute -> fixed
- joint gripper_right_inner_finger_joint: type revolute -> fixed
- joint gripper_right_inner_knuckle_joint: type revolute -> fixed
